File: pcb/supplyAndReceiver5Vold/receiver.kicad_pcb (KiCad board)
At the start: 2 copper layers, 20 x 16 mm, 7 parts, among them J1 WAGO 2061-602, J2 har-flexicon 2,54 MSH-4, J3 Conn_01x05_Socket, J4 Conn_01x02, U1 SP485CN

Commit message: Use ISL3280E
Parts:
- C1: footprint Capacitor_SMD:C_0603_1608Metric -> local:0603
- J4: value Conn_01x02 -> Kyocera-009176002001906
- R1: footprint Resistor_SMD:R_1206_3216Metric -> local:1206
- U1: footprint local:SP485 -> local:SO-8
