File: pcb/supplyAndReceiver5Vold/receiver.kicad_sch (KiCad schematic)
At the start: 7 parts, among them J1 Conn_01x05_Socket, J1 WAGO 2061-602, J2 har-flexicon 2,54 MSH-4, J4 Kyocera-009176002001906, U1 SP485CN

Commit message: Use ISL3280E
Parts:
- C1: footprint Capacitor_SMD:C_0603_1608Metric -> local:0603
- R1: footprint Resistor_SMD:R_1206_3216Metric -> local:1206; now not fitted
- U1: footprint local:SP485 -> local:SO-8
