File: pcb/longSupplyAndReceiver5V/receiver.kicad_sch (KiCad schematic)
At the start: 7 parts, among them J1 Conn_01x05_Socket, J1 WAGO 2061-602, J2 har-flexicon 2,54 MSH-4, J4 Kyocera-009176002001906, U1 SP485CN

Commit message: New pin ordering for Harting connector
Parts:
- removed U1: SP485CN, local:SO-8, symbol Interface_UART:SP3485CN
- added U1: ISL3281E, local:ISL3281E, symbol Interface_UART:ISL3281ExHZ
- C1: footprint local:0603 -> Capacitor_SMD:C_0603_1608Metric
- J1: footprint local:HolesL -> local:SolderHoles3pin10mm
- R1: footprint local:1206 -> Resistor_SMD:R_1206_3216Metric
Connections:
- net +15V: now also J2.2 (Pin_2); no longer J2.3 (Pin_3)
- net +5V: now also U1.1 (VCC), U1.5 (RE)
- net DATA: now also U1.3 (RO)
- net GND: now also J2.1 (Pin_1), U1.2 (GND); no longer J2.4 (Pin_4)
- net RS485_A: now also J2.3 (Pin_3), U1.6 (A); no longer J2.2 (Pin_2)
- net RS485_B: now also J2.4 (Pin_4), U1.4 (B); no longer J2.1 (Pin_1)
Other:
- note added: "RS485 receiver ISL3280E / ISL3281E / MAX3280E / MAX3281E"
- moved on the sheet: J1, J2, R1
