File: pcb/metodReceiver12V/receiver.kicad_pcb (KiCad board)
At the start: 2 copper layers, 300 x 48 mm, 22 parts, among them J1 WAGO 2061-602, J2 har-flexicon 2,54 MSH-4, J3 Conn_01x05_Socket, J4 Conn_01x05_Socket, J5 Conn_01x05_Socket, J6 Conn_01x05_Socket, U1 TLV76050, U2 ISL3280ExHZ, U3 TLV76050, U4 ISL3280ExHZ

Commit message: Use ISL3280E
Parts:
- C1, C2, C3, C4: footprint Capacitor_SMD:C_0603_1608Metric -> local:0603
- J5 (x2), J6 (x2): footprint local:LedConnector -> local:LedConnector3pin10mm
- R1, R2: footprint Resistor_SMD:R_1206_3216Metric -> local:1206
- U1, U3: value TLV76050 -> TLV76050DBZ
- U2, U4: value ISL3280ExHZ -> ISL3281E; footprint local:ISL3280E -> local:ISL3281E
- turned U1 to -90 degrees
- turned U3 to 90 degrees
Connections:
- J5 pad 1: (no net) -> Net-(J5-Pin_1) (x2)
- J5 pad 2: (no net) -> Net-(J5-Pin_2) (x2)
- J5 pad 3: (no net) -> Net-(J5-Pin_3) (x2)
- J6 pad 1: (no net) -> Net-(J5-Pin_1) (x2)
- J6 pad 2: (no net) -> Net-(J5-Pin_2) (x2)
- J6 pad 3: (no net) -> Net-(J5-Pin_3) (x2)
- U2 pad 5: RS485_A -> +5V_A
- U4 pad 5: RS485_A -> +5V_B
Routing:
- net (no net): track 183.6 -> 0.00 mm
- net Net-(J5-Pin_2): track 42.3 -> 132.3 mm
- net Net-(J5-Pin_1): track 26.9 -> 82.6 mm
- net Net-(J5-Pin_3): track 17.4 -> 55.3 mm
- net +5V_A: track 8.45 -> 11.2 mm
- net +5V_B: track 4.30 -> 6.48 mm
Other:
- outline, holes or cut-outs redrawn
- board text added: "Board"

Commit message: New pin ordering for Harting connector
Parts:
- moved J5 28.0 mm to (208.0, 116.5)
- moved J6 28.0 mm to (223.0, 118.5)
- moved J5 14.0 mm to (234.0, 117.5)
- moved J6 14.0 mm to (249.0, 118.5)
- turned J2 to 180 degrees
Routing:
- net +12V: track 82.8 -> 64.6 mm
- net RS485_B: track 304.0 -> 299.8 mm
- net RS485_A: track 301.4 -> 300.1 mm
- net GND: track 87.2 -> 87.8 mm
Other:
- outline, holes or cut-outs redrawn
