File: pcb/Regulator30Leds17V5V/Regulator30Leds17V5V.kicad_pcb (KiCad board)
At the start: 4 copper layers, 33.3 x 20 mm, 17 parts, among them J1 Conn_01x02, J2 Conn_01x05_Socket, J3 Conn_01x05_Socket, U1 TPS82130, U2 TPS82130

Commit message: Minor changes
Parts:
- moved JP1 4.00 mm to (131.0, 108.5)
Routing:
- net GND: track 10.9 -> 11.6 mm
Changed lines of the file:
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@@
 		(sheetname "/")
 		(sheetfile "Regulator30Leds17V5V.kicad_sch")
-		(units
-			(unit
-				(name "A")
-				(pins "1" "2" "3")
-			)
-		)
 		(solder_mask_margin 0)
 		(solder_paste_margin 0)
@@
 		(sheetname "/")
 		(sheetfile "Regulator30Leds17V5V.kicad_sch")
-		(units
-			(unit
-				(name "A")
-				(pins "1" "2")
-			)
-		)
 		(solder_mask_margin 0)
 		(solder_paste_margin 0)
@@
 		(sheetname "/")
 		(sheetfile "Regulator30Leds17V5V.kicad_sch")
-		(units
-			(unit
-				(name "A")
-				(pins "1" "2")
-			)
-		)
 		(solder_mask_margin 0)
 		(solder_paste_margin 0)
@@
 		(sheetname "/")
 		(sheetfile "Regulator30Leds17V5V.kicad_sch")
-		(units
-			(unit
-				(name "A")
-				(pins "2" "1" "7" "8" "3" "9" "4" "5" "6")
-			)
-		)
 		(solder_mask_margin 0)
 		(solder_paste_margin 0)
@@
 		(sheetname "/")
 		(sheetfile "Regulator30Leds17V5V.kicad_sch")
-		(units
-			(unit
-				(name "A")
-				(pins "1" "2")
-			)
-		)
 		(solder_mask_margin 0)
 		(solder_paste_margin 0)
@@
 		(sheetname "/")
 		(sheetfile "Regulator30Leds17V5V.kicad_sch")
-		(units
-			(unit
-				(name "A")
-				(pins "1" "2")
-			)
-		)
 		(solder_mask_margin 0)
 		(solder_paste_margin 0)
@@
 		(sheetname "/")
 		(sheetfile "Regulator30Leds17V5V.kicad_sch")
-		(units
-			(unit
-				(name "A")
-				(pins "1" "2")
-			)
-		)
 		(solder_mask_margin 0)
 		(solder_paste_margin 0)
@@
 		(sheetname "/")
 		(sheetfile "Regulator30Leds17V5V.kicad_sch")
-		(units
-			(unit
-				(name "A")
-				(pins "2" "1" "7" "8" "3" "9" "4" "5" "6")
-			)
-		)
 		(solder_mask_margin 0)
 		(solder_paste_margin 0)
@@
 	(footprint "local:Jumper"
 		(layer "F.Cu")
-		(at 135 108.5)
+		(at 131 108.5)
 		(descr "Jumper with 2 pads and 0.15mm gap")
 		(property "Reference" "JP1"
@@
 		(sheetname "/")
 		(sheetfile "Regulator30Leds17V5V.kicad_sch")
-		(units
-			(unit
-				(name "A")
-				(pins "1" "2")
-			)
-		)
 		(solder_mask_margin 0)
 		(solder_paste_margin 0)
@@
 		(sheetname "/")
 		(sheetfile "Regulator30Leds17V5V.kicad_sch")
-		(units
-			(unit
-				(name "A")
-				(pins "1" "2" "3")
-			)
-		)
 		(solder_mask_margin 0)
 		(solder_paste_margin 0)
@@
 		(sheetname "/")
 		(sheetfile "Regulator30Leds17V5V.kicad_sch")
-		(units
-			(unit
-				(name "A")
-				(pins "1" "2")
-			)
-		)
 		(solder_mask_margin 0)
 		(solder_paste_margin 0)
@@
 		(sheetname "/")
 		(sheetfile "Regulator30Leds17V5V.kicad_sch")
-		(units
-			(unit
-				(name "A")
-				(pins "1" "2")
-			)
-		)
 		(solder_mask_margin 0)
 		(solder_paste_margin 0)
@@
 		(sheetname "/")
 		(sheetfile "Regulator30Leds17V5V.kicad_sch")
-		(units
-			(unit
-				(name "A")
-				(pins "1" "2")
-			)
-		)
 		(solder_mask_margin 0)
 		(solder_paste_margin 0)
@@
 		(sheetname "/")
 		(sheetfile "Regulator30Leds17V5V.kicad_sch")
-		(units
-			(unit
-				(name "A")
-				(pins "4" "1" "3" "2")
-			)
-		)
 		(solder_mask_margin 0)
 		(solder_paste_margin 0)
@@
 		)
 		(fp_line
+			(start 0.1 2.65)
+			(end 2.65 0.1)
+			(stroke
+				(width 0.15)
+				(type solid)
+			)
+			(layer "F.SilkS")
+		)
+		(fp_line
 			(start -2.575 -2.575)
 			(end -2.725 -2.575)
@@
 		(sheetname "/")
 		(sheetfile "Regulator30Leds17V5V.kicad_sch")
-		(units
-			(unit
-				(name "A")
-				(pins "1" "2")
-			)
-		)
 		(solder_mask_margin 0)
 		(solder_paste_margin 0)
@@
 		(sheetname "/")
 		(sheetfile "Regulator30Leds17V5V.kicad_sch")
-		(units
-			(unit
-				(name "A")
-				(pins "1" "2")
-			)
-		)
 		(solder_mask_margin 0)
 		(solder_paste_margin 0)
@@
 		(sheetname "/")
 		(sheetfile "Regulator30Leds17V5V.kicad_sch")
-		(units
-			(unit
-				(name "A")
-				(pins "1" "2")
-			)
-		)
 		(solder_mask_margin 0)
 		(solder_paste_margin 0)
@@
 	)
 	(segment
+		(start 141.8 106.25)
+		(end 142.5 106.25)
+		(width 0.4)
+		(layer "F.Cu")
+		(net "GND")
+	)
+	(segment
 		(start 123 106.25)
 		(end 123.15 106.25)
@@
 		(polygon
 			(pts
-				(xy 135.25 106.75) (xy 135.25 109) (xy 150.5 109) (xy 150.5 106.75)
+				(xy 131.1 106.75) (xy 131.1 109) (xy 150.5 109) (xy 150.5 106.75)
 			)
 		)
@@
 		(polygon
 			(pts
-				(xy 119 106.75) (xy 119 109) (xy 134.75 109) (xy 134.75 106.75)
+				(xy 119 106.75) (xy 119 109) (xy 130.9 109) (xy 130.9 106.75)
 			)
 		)
